Commit message: Change urdf to add AR tag transformation for calibration

File: jenga_ur5_control/urdf/ur5_with_jenga_tool.xacro (robot description, xacro)
@@ -63,4 +63,5 @@
   </link>
   <link name="tool_range_finder" />
+  <link name="tool_ar_tag" />
   <joint name="jenga_tool_to_gripper" type="fixed">
     <axis xyz="0 0 0" />
@@ -81,3 +82,9 @@
     <child link="tool_range_finder" />
   </joint>
+  <joint name="jenga_tool_to_ar_tag" type="fixed">
+    <axis xyz="0 0 0" />
+    <origin xyz="0 0.02933 0.0275" rpy="${-pi/2} 0 0" />
+    <parent link="jenga_tool" />
+    <child link="tool_ar_tag" />
+  </joint>
 </robot>

Commit message: Modify ar tag location to add some white space around the tag

File: jenga_ur5_control/urdf/ur5_with_jenga_tool.xacro (robot description, xacro)
@@ -84,5 +84,5 @@
   <joint name="jenga_tool_to_ar_tag" type="fixed">
     <axis xyz="0 0 0" />
-    <origin xyz="0 0.02933 0.0275" rpy="${-pi/2} 0 0" />
+    <origin xyz="0 0.02763 0.0325" rpy="${-pi/2} 0 0" />
     <parent link="jenga_tool" />
     <child link="tool_ar_tag" />

Commit message: Further polishing

File: jenga_ur5_control/urdf/ur5_with_jenga_tool.xacro (robot description, xacro)
@@ -78,5 +78,5 @@
   <joint name="jenga_tool_to_range_finder" type="fixed">
     <axis xyz="0 0 0" />
-    <origin xyz="0 -0.02942 0.059234" rpy="0 0 0" />
+    <origin xyz="0 -0.02642 0.059234" rpy="0 0 0" />
     <parent link="jenga_tool" />
     <child link="tool_range_finder" />

Commit message: Start implementing range finder compensation

File: jenga_ur5_control/urdf/ur5_with_jenga_tool.xacro (robot description, xacro)
@@ -72,5 +72,5 @@
   <joint name="jenga_tool_to_probe" type="fixed">
     <axis xyz="0 0 0" />
-    <origin xyz="0.0795 0 0.026146" rpy="0 ${pi/2} 0" />
+    <origin xyz="0.0795 -0.003 0.016146" rpy="0 ${pi/2} 0" />
     <parent link="jenga_tool" />
     <child link="tool_probe" />
@@ -78,5 +78,5 @@
   <joint name="jenga_tool_to_range_finder" type="fixed">
     <axis xyz="0 0 0" />
-    <origin xyz="0 -0.02642 0.059234" rpy="0 0 0" />
+    <origin xyz="0 -0.02642 0.039234" rpy="0 0 0" />
     <parent link="jenga_tool" />
     <child link="tool_range_finder" />

Commit message: Modify xacro for range finder frame

File: jenga_ur5_control/urdf/ur5_with_jenga_tool.xacro (robot description, xacro)
@@ -78,5 +78,5 @@
   <joint name="jenga_tool_to_range_finder" type="fixed">
     <axis xyz="0 0 0" />
-    <origin xyz="0 -0.02642 0.039234" rpy="0 0 0" />
+    <origin xyz="0 -0.02642 0.059234" rpy="0 0 0" />
     <parent link="jenga_tool" />
     <child link="tool_range_finder" />

Commit message: Implement and tested initialization code

File: jenga_ur5_control/urdf/ur5_with_jenga_tool.xacro (robot description, xacro)
@@ -66,5 +66,5 @@
   <joint name="jenga_tool_to_gripper" type="fixed">
     <axis xyz="0 0 0" />
-    <origin xyz="0 0 0.072646" rpy="0 0 0" />
+    <origin xyz="0 0 0.077646" rpy="0 0 0" />
     <parent link="jenga_tool" />
     <child link="tool_gripper" />

Commit message: Further tuning to have the robot play at a slower speed

File: jenga_ur5_control/urdf/ur5_with_jenga_tool.xacro (robot description, xacro)
@@ -72,5 +72,5 @@
   <joint name="jenga_tool_to_probe" type="fixed">
     <axis xyz="0 0 0" />
-    <origin xyz="0.0795 -0.003 0.016146" rpy="0 ${pi/2} 0" />
+    <origin xyz="0.0795 -0.003 0.026146" rpy="0 ${pi/2} 0" />
     <parent link="jenga_tool" />
     <child link="tool_probe" />
